File: hardware/dist/circuit_fuzz.kicad_sch (KiCad schematic)
At the start: 46 parts, among them Q1 BC547B, Q2 BC547B, U8 TL072

Commit message: bom + kicad fix for dual supply
Parts:
- removed C34, C44: 22n, symbol Device:C
- removed R35, R53: 1M, symbol Device:R
- C35, C37, C38, C40, C42, C45, C46: footprint (none) -> Capacitor_SMD:C_0402_1005Metric
- C36: value 22n -> 1u; footprint (none) -> Capacitor_SMD:C_0402_1005Metric
- C39, C41: footprint (none) -> Capacitor_THT:CP_Radial_D4.0mm_P1.50mm
- C43: value 4n -> 4.7n; footprint (none) -> Capacitor_SMD:C_0402_1005Metric
- D5, D6, D7, D8: footprint Diode_THT:D_DO-35_SOD27_P7.62mm_Horizontal -> Diode_SMD:D_SOD-323
- R33: value 20k -> 200k; footprint (none) -> Resistor_SMD:R_0402_1005Metric
- R34: value 10k -> 100k; footprint (none) -> Resistor_SMD:R_0402_1005Metric
- R36, R37, R38, R39, R40, R41, R42, R43, R44, R45, R46, R47, R48, R49, R50, R51, R52, R55: footprint (none) -> Resistor_SMD:R_0402_1005Metric
- R54: value 40k -> 150k; footprint (none) -> Resistor_SMD:R_0402_1005Metric
- RV10, RV8, RV9: footprint (none) -> Potentiometer_THT:Potentiometer_Alps_RK09K_Single_Vertical
- U4, U5: renamed from U8; footprint (none) -> TL072CDT:D8_TEX_STM
Connections:
- net BIAS is gone; now on net GND: R52.1, RV10.3
- net at C46.1, R54.2: now also U5.1; no longer U5.7
- net at R52.2, R54.1: now also U5.2 (-); no longer U5.6 (-)
- net at C36.1, R37.1: now also U4.7; no longer U4.1
- net at R37.2, R38.1: now also U4.6 (-); no longer U4.2 (-)
- net at RV9.2: now also U5.3 (+)
- net at C35.2, R36.1: now also U4.5 (+); no longer U4.3 (+)
- net at R36.2: now also R33.2, R34.2
Other:
- moved on the sheet: R33, R34

Commit message: finish pcb
Parts:
- C35, C36, C37, C38, C40, C42, C43, C45, C46: footprint Capacitor_SMD:C_0402_1005Metric -> Capacitor_SMD:C_0805_2012Metric_Pad1.18x1.45mm_HandSolder
- R33, R34, R36, R37, R38, R39, R40, R41, R42, R43, R44, R45, R46, R47, R48, R49, R50, R51, R52, R54, R55: footprint Resistor_SMD:R_0402_1005Metric -> Resistor_SMD:R_0805_2012Metric_Pad1.20x1.40mm_HandSolder
- renumbered U4 to U5
Connections:
- net at C46.1, R54.2: now also U5.7; no longer U5.1
- net at R52.2, R54.1: now also U5.6 (-); no longer U5.2 (-)
- net at RV9.2: now also U5.5 (+); no longer U5.3 (+)
- net at C36.1, R37.1: now also U5.1; no longer U5.7
- net at R37.2, R38.1: now also U5.2 (-); no longer U5.6 (-)
- net at C35.2, R36.1: now also U5.3 (+); no longer U5.5 (+)
- net VDD renamed +12V
