File: hardware/dist/circuit_wrmergle.kicad_sch (KiCad schematic)
At the start: 48 parts, among them Q3 BC547B, Q4 BC547B, Q5 BSP89, U6 TL072, U9 TL072

Commit message: bom + kicad fix for dual supply
Parts:
- removed C47, C59: 22n, symbol Device:C
- removed R58, R74: 1M, symbol Device:R
- C48: value 220n -> 100n; footprint (none) -> Capacitor_SMD:C_0402_1005Metric
- C49, C50, C51, C54, C58, C60: footprint (none) -> Capacitor_SMD:C_0402_1005Metric
- C52, C53, C55, C56: footprint (none) -> Capacitor_THT:CP_Radial_D4.0mm_P1.50mm
- C57: value 4n -> 4.7n; footprint (none) -> Capacitor_SMD:C_0402_1005Metric
- D10, D11, D12, D9: footprint Diode_THT:D_DO-35_SOD27_P7.62mm_Horizontal -> Diode_SMD:D_SOD-323
- R56: value 20k -> 200k; footprint (none) -> Resistor_SMD:R_0402_1005Metric
- R57: value 10k -> 100k; footprint (none) -> Resistor_SMD:R_0402_1005Metric
- R59: value 5k -> 10k; footprint (none) -> Resistor_SMD:R_0402_1005Metric
- R60, R61, R62, R63, R65, R66, R67, R68, R69, R70, R71, R72, R73, R75, R76: footprint (none) -> Resistor_SMD:R_0402_1005Metric
- R64: value 2.2M -> 1M; footprint (none) -> Resistor_SMD:R_0402_1005Metric
- RV11, RV12, RV13: footprint (none) -> Potentiometer_THT:Potentiometer_Alps_RK09K_Single_Vertical
- RV14: footprint (none) -> Connector_PinHeader_2.54mm:PinHeader_1x03_P2.54mm_Vertical
- U6: renamed from U9; footprint (none) -> TL072CDT:D8_TEX_STM
- U7: renamed from U6; footprint (none) -> TL072CDT:D8_TEX_STM
Connections:
- net BIAS is gone; now on net GND: R57.1, R73.1, RV11.1, RV14.3
- net at C48.1: now also R56.2, R57.2
- net at C60.1, R75.2: now also U7.1; no longer U7.7
- net at R73.2, R75.1: now also U7.2 (-); no longer U7.6 (-)
- net at RV13.2: now also U7.3 (+)
Other:
- moved on the sheet: R56, R57

Commit message: finish pcb
Parts:
- C48, C49, C50, C51, C54, C57, C58, C60: footprint Capacitor_SMD:C_0402_1005Metric -> Capacitor_SMD:C_0805_2012Metric_Pad1.18x1.45mm_HandSolder
- R56, R57, R59, R60, R61, R62, R63, R65, R66, R67, R68, R69, R70, R71, R72, R73, R75, R76: footprint Resistor_SMD:R_0402_1005Metric -> Resistor_SMD:R_0805_2012Metric_Pad1.20x1.40mm_HandSolder
- R64: value 1M -> 2.2M; footprint Resistor_SMD:R_0402_1005Metric -> Resistor_SMD:R_0805_2012Metric_Pad1.20x1.40mm_HandSolder
- RV12: footprint Potentiometer_THT:Potentiometer_Alps_RK09K_Single_Vertical -> 3362P-1-253LF:TRIM_3362P-1-253LF
- RV14: footprint Connector_PinHeader_2.54mm:PinHeader_1x03_P2.54mm_Vertical -> Potentiometer_THT:Potentiometer_Alps_RK09K_Single_Vertical
Connections:
- net at Q3.2 (B), R64.2: now also C52.2; no longer C52.1
- net at RV12.3: now also C52.1; no longer C52.2
- net VDD renamed +12V
Other:
- moved on the sheet: C52
